File: eda/lumi-square/LumiSquare.kicad_sch (KiCad schematic)
At the start: 89 parts, among them J1 USB_C_Receptacle_USB2.0_14P, J2 Conn_01x12, J3 Conn_01x12, J4 Conn_ARM_JTAG_SWD_10, J5 Conn_01x08, J6 Conn_01x08, Q1 IRLML6244, Q10 IRLML2246, Q2 IRLML2246, Q3 IRLML2246, Q4 MMBT3904, Q5 MMBT3904, Q6 MMBT3904, Q7 MMBT3904, Q8 MMBT3904, Q9 MMBT3904, SW1 SW_SPST, SW2 SW_Push, SW3 SW_Push, SW4 SW_Push, SW5 SW_Push, U1 MCP73831-2-OT, U2 TPS3840, U3 TLV61070A, U4 TLV61070A, U5 ATSAMD21J18A-A, U6 STP16CPC05MTR, U8 MIC5225-3.3YM5

Commit message: -Added circuity for esd on usb. - Add p chanel mosfets. - added new footprint, symbol, and step files
Parts:
- removed J4: Conn_ARM_JTAG_SWD_10, symbol Connector:Conn_ARM_JTAG_SWD_10
- added J7: FTSH-105-01-X-DV-P-K-X, FTSH-105-01-X-DV-P-K-X:SAMTEC_FTSH-105-01-X-DV-P-K-X, symbol FTSH-105-01-X-DV-P-K-X:FTSH-105-01-X-DV-P-K-X
- added Q15, Q16, Q17, Q18: TSM680P06CH, TSM680P06CH:TO228P680X245X847-3, symbol TSM680P06CH:TSM680P06CH
- added R29, R31, R33, R35: 100k, Resistor_SMD:R_0603_1608Metric_Pad0.98x0.95mm_HandSolder, symbol Device:R_US
- added R30, R32, R34, R36: 47k, Resistor_SMD:R_0603_1608Metric_Pad0.98x0.95mm_HandSolder, symbol Device:R_US
- added U7: CM1224-02SR, CM1224-02SR:SOT143, symbol CM1224-02SR:CM1224-02SR
- C13, C14, C15: footprint Capacitor_THT:CP_Radial_D6.3mm_P2.50mm -> Capacitor_SMD:C_0201_0603Metric_Pad0.64x0.40mm_HandSolder
- C16, C17, C18, C19, C20, C21: footprint Capacitor_SMD:C_1206_3216Metric -> Capacitor_SMD:C_0201_0603Metric_Pad0.64x0.40mm_HandSolder
- R12: value 1k -> 200
- SW1, SW2, SW3, SW4: footprint (none) -> Connector_PinHeader_2.54mm:PinHeader_1x02_P2.54mm_Vertical
- SW5: footprint (none) -> Button_Switch_THT:SW_TH_Tactile_Omron_B3F-100x
Connections:
- net +3.3V Main: now also J7.01
- net 5.3V Out: now also Q15.3, Q16.3, Q17.3, Q18.3, R29.2, R31.2, R33.2, R35.2; no longer Q4.3 (C), Q5.3 (C), Q6.3 (C), Q7.3 (C)
- net 5V USB: now also U7.4 (VP)
- net GNDREF: now also Q4.2 (E), Q5.2 (E), Q6.2 (E), Q7.2 (E), J7.03, J7.05, J7.09, R30.1, R32.1, R34.1, R36.1, U7.1 (VN)
- net Reset Pin: now also J7.10
- net SWCLK: now also J7.04
- net SWDIO: now also J7.02
- net at Q4.1 (B), R16.2: now also R30.2
- net Col 1 Anode: now reaches J3.9 (Pin_9)
- net Col 1 Anode: now also Q15.2; no longer Q4.2 (E)
- net at Q5.1 (B), R17.2: now also R32.2
- net Col 2 Anode: now reaches J3.10 (Pin_10)
- net Col 2 Anode: now also Q17.2; no longer Q5.2 (E)
- net Col 3 Anode: now reaches J3.11 (Pin_11)
- net Col 3 Anode: now also Q16.2; no longer Q6.2 (E)
- net Col 4 Anode: now reaches J3.12 (Pin_12)
- net Col 4 Anode: now also Q18.2; no longer Q7.2 (E)
- net at Q6.1 (B), R18.2: now also R34.2
- net TARGET USB N: now reaches U5.45 (PA24)
- net TARGET USB N: now also J1.A7 (D-), J1.B7 (D-), U7.3 (CH2)
- net TARGET USB P: now reaches U5.46 (PA25)
- net TARGET USB P: now also J1.A6 (D+), J1.B6 (D+), U7.2 (CH1)
- net at Q7.1 (B), R19.2: now also R36.2
- new net: Q15.1, Q4.3 (C), R29.1
- new net: Q17.1, Q5.3 (C), R31.1
- new net: Q16.1, Q6.3 (C), R33.1
- new net: Q18.1, Q7.3 (C), R35.1
Other:
- moved on the sheet: C11, C12, J2, J3, Q4, Q5, Q6, Q7, R12, R16, R17, R18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

Commit message: Adding updateds to pcb and schematic design
Parts:
- removed BZ1: Buzzer, symbol Device:Buzzer
- removed J5, J6: Conn_01x08, Connector_PinSocket_2.54mm:PinSocket_1x08_P2.54mm_Vertical, symbol Connector_Generic:Conn_01x08
- added BZ2: RDT-4.000-1375-NS1, RDT.pretty:RDT-4.000-1375-NS1, symbol RDT-4.000-1375-NS1:RDT-4.000-1375-NS1
- added U9: DFR0299, DFR0299:MODULE_DFR0299, symbol DFR0299:DFR0299
- C13, C14, C15, C16, C17, C18, C19, C20, C21: footprint Capacitor_SMD:C_0201_0603Metric_Pad0.64x0.40mm_HandSolder -> Capacitor_SMD:C_0603_1608Metric_Pad1.08x0.95mm_HandSolder
Connections:
- net +3.3V Main: now also BZ2.1 (+), U9.1 (VCC)
- net MCU RX: now also U9.3 (TX)
- net MCU TX: now also U9.2 (RX)
- net Speaker+: now also U9.6 (SPK1)
- net Speaker-: now also U9.8 (SPK2)
- net at D4.2 (A), Q8.3 (C): now also BZ2.2 (-)
- net GNDREF renamed GND
- net GND: now also U9.10 (GND), U9.7 (GND)
Other:
- moved on the sheet: D4, Q8, R22

Commit message: Made more progress with the pcb layout
Parts:
- added J4: Conn_01x02, Connector_JST:JST_SH_BM02B-SRSS-TB_1x02-1MP_P1.00mm_Vertical, symbol Connector_Generic:Conn_01x02
- D1, D5: footprint LED_SMD:LED_1206_3216Metric -> Connector_JST:JST_SH_BM02B-SRSS-TB_1x02-1MP_P1.00mm_Vertical
- SW1, SW2, SW3, SW4: footprint Connector_PinHeader_2.54mm:PinHeader_1x02_P2.54mm_Vertical -> Connector_JST:JST_SH_BM02B-SRSS-TB_1x02-1MP_P1.00mm_Vertical
- SW5: footprint Button_Switch_THT:SW_TH_Tactile_Omron_B3F-100x -> Button_Switch_SMD:SW_SPST_TL3342
- renumbered C23234545 to C22, C3245345 to C23
Connections:
- net Speaker+: now also J4.1 (Pin_1)
- net Speaker-: now also J4.2 (Pin_2)
Changed lines of the file:
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@@
 	)
 	(junction
+		(at 176.53 189.23)
+		(diameter 0)
+		(color 0 0 0 0)
+	)
+	(junction
 		(at 570.23 213.36)
 		(diameter 0)
@@
 	)
 	(junction
+		(at 176.53 191.77)
+		(diameter 0)
+		(color 0 0 0 0)
+	)
+	(junction
 		(at 391.16 222.25)
 		(diameter 0)
@@
 	(wire
 		(pts
+			(xy 173.99 189.23) (xy 176.53 189.23)
+		)
+		(stroke
+			(width 0)
+			(type default)
+		)
+	)
+	(wire
+		(pts
 			(xy 68.58 55.88) (xy 68.58 57.15)
 		)
@@
 	(wire
 		(pts
-			(xy 173.99 189.23) (xy 177.8 189.23)
-		)
-		(stroke
-			(width 0)
-			(type default)
-		)
-	)
-	(wire
-		(pts
 			(xy 557.53 227.33) (xy 552.45 227.33)
 		)
@@
 	(wire
 		(pts
+			(xy 176.53 191.77) (xy 177.8 191.77)
+		)
+		(stroke
+			(width 0)
+			(type default)
+		)
+	)
+	(wire
+		(pts
 			(xy 38.1 73.66) (xy 38.1 81.28)
 		)
@@
 	(wire
 		(pts
+			(xy 176.53 191.77) (xy 176.53 200.66)
+		)
+		(stroke
+			(width 0)
+			(type default)
+		)
+	)
+	(wire
+		(pts
 			(xy 401.32 173.99) (xy 401.32 175.26)
 		)
@@
 	(wire
 		(pts
-			(xy 173.99 191.77) (xy 177.8 191.77)
-		)
-		(stroke
-			(width 0)
-			(type default)
-		)
-	)
-	(wire
-		(pts
 			(xy 194.31 255.27) (xy 214.63 255.27)
 		)
@@
 	(wire
 		(pts
+			(xy 173.99 191.77) (xy 176.53 191.77)
+		)
+		(stroke
+			(width 0)
+			(type default)
+		)
+	)
+	(wire
+		(pts
 			(xy 55.88 48.26) (xy 53.34 48.26)
 		)
@@
 	(wire
 		(pts
+			(xy 172.72 185.42) (xy 176.53 185.42)
+		)
+		(stroke
+			(width 0)
+			(type default)
+		)
+	)
+	(wire
+		(pts
 			(xy 480.06 162.56) (xy 486.41 162.56)
 		)
@@
 	(wire
 		(pts
+			(xy 176.53 185.42) (xy 176.53 189.23)
+		)
+		(stroke
+			(width 0)
+			(type default)
+		)
+	)
+	(wire
+		(pts
 			(xy 278.13 33.02) (xy 287.02 33.02)
 		)
@@
 	(wire
 		(pts
+			(xy 173.99 200.66) (xy 176.53 200.66)
+		)
+		(stroke
+			(width 0)
+			(type default)
+		)
+	)
+	(wire
+		(pts
 			(xy 59.69 35.56) (xy 83.82 35.56)
 		)
@@
 	(wire
 		(pts
+			(xy 176.53 189.23) (xy 177.8 189.23)
+		)
+		(stroke
+			(width 0)
+			(type default)
+		)
+	)
+	(wire
+		(pts
 			(xy 308.61 49.53) (xy 308.61 54.61)
 		)
@@
 	)
 	(label "Speaker+"
-		(at 173.99 189.23 180)
+		(at 172.72 185.42 180)
 		(effects
 			(font
@@
 	)
 	(label "Speaker-"
-		(at 173.99 191.77 180)
+		(at 173.99 200.66 180)
 		(effects
 			(font
@@
 		(dnp no)
 		(fields_autoplaced yes)
-		(property "Reference" "C3245345"
+		(property "Reference" "C23"
 			(at 506.73 91.4399 0)
 			(show_name no)
@@
 			(project "LumiSquare"
 				(path "/092b428a-5a5f-4f13-b55d-abd406e11b5b"
-					(reference "C3245345")
+					(reference "C23")
 					(unit 1)
 				)
@@
 			)
 		)
-		(property "Footprint" "LED_SMD:LED_1206_3216Metric"
+		(property "Footprint" "Connector_JST:JST_SH_BM02B-SRSS-TB_1x02-1MP_P1.00mm_Vertical"
 			(at 134.62 58.42 0)
 			(hide yes)
@@
 			)
 		)
-		(property "Footprint" "Connector_PinHeader_2.54mm:PinHeader_1x02_P2.54mm_Vertical"
+		(property "Footprint" "Connector_JST:JST_SH_BM02B-SRSS-TB_1x02-1MP_P1.00mm_Vertical"
 			(at 457.2 157.48 0)
 			(hide yes)
@@
 			)
 		)
-		(property "Footprint" "Button_Switch_THT:SW_TH_Tactile_Omron_B3F-100x"
+		(property "Footprint" "Button_Switch_SMD:SW_SPST_TL3342"
 			(at 459.74 222.25 0)
 			(hide yes)
@@
 			)
 		)
-		(property "Footprint" "Connector_PinHeader_2.54mm:PinHeader_1x02_P2.54mm_Vertical"
+		(property "Footprint" "Connector_JST:JST_SH_BM02B-SRSS-TB_1x02-1MP_P1.00mm_Vertical"
 			(at 453.39 87.63 0)
 			(hide yes)
@@
 		(dnp no)
 		(fields_autoplaced yes)
-		(property "Reference" "C23234545"
+		(property "Reference" "C22"
 			(at 478.79 91.4399 0)
 			(show_name no)
@@
 			(project "LumiSquare"
 				(path "/092b428a-5a5f-4f13-b55d-abd406e11b5b"
-					(reference "C23234545")
+					(reference "C22")
 					(unit 1)
 				)
@@
 	)
 	(symbol
+		(lib_id "Connector_Generic:Conn_01x02")
+		(at 168.91 189.23 0)
+		(mirror y)
+		(unit 1)
+		(body_style 1)
+		(exclude_from_sim no)
+		(in_bom yes)
+		(on_board yes)
+		(in_pos_files yes)
+		(dnp no)
+		(property "Reference" "J4"
+			(at 166.37 189.2299 0)
+			(show_name no)
+			(do_not_autoplace no)
+			(effects
+				(font
+					(size 1.27 1.27)
+				)
+				(justify left)
+			)
+		)
+		(property "Value" "Conn_01x02"
+			(at 175.006 195.834 0)
+			(show_name no)
+			(do_not_autoplace no)
+			(effects
+				(font
+					(size 1.27 1.27)
+				)
+				(justify left)
+			)
+		)
+		(property "Footprint" "Connector_JST:JST_SH_BM02B-SRSS-TB_1x02-1MP_P1.00mm_Vertical"
+			(at 168.91 189.23 0)
+			(hide yes)
+			(show_name no)
+			(do_not_autoplace no)
+			(effects
+				(font
+					(size 1.27 1.27)
+				)
+			)
+		)
+		(property "Datasheet" ""
+			(at 168.91 189.23 0)
+			(hide yes)
+			(show_name no)
+			(do_not_autoplace no)
+			(effects
+				(font
+					(size 1.27 1.27)
+				)
+			)
+		)
+		(property "Description" "Generic connector, single row, 01x02, script generated (kicad-library-utils/schlib/autogen/connector/)"
+			(at 168.91 189.23 0)
+			(hide yes)
+			(show_name no)
+			(do_not_autoplace no)
+			(effects
+				(font
+					(size 1.27 1.27)
+				)
+			)
+		)
+		(pin "1"
+		)
+		(pin "2"
+		)
+		(instances
+			(project "LumiSquare"
+				(path "/092b428a-5a5f-4f13-b55d-abd406e11b5b"
+					(reference "J4")
+					(unit 1)
+				)
+			)
+		)
+	)
+	(symbol
 		(lib_id "power:GNDREF")
 		(at 491.49 109.22 0)
@@
 			)
 		)
-		(property "Footprint" "LED_SMD:LED_1206_3216Metric"
+		(property "Footprint" "Connector_JST:JST_SH_BM02B-SRSS-TB_1x02-1MP_P1.00mm_Vertical"
 			(at 523.24 102.87 0)
 			(hide yes)
@@
 			)
 		)
-		(property "Footprint" "Connector_PinHeader_2.54mm:PinHeader_1x02_P2.54mm_Vertical"
+		(property "Footprint" "Connector_JST:JST_SH_BM02B-SRSS-TB_1x02-1MP_P1.00mm_Vertical"
 			(at 378.46 157.48 0)
 			(hide yes)
@@
 			)
 		)
-		(property "Footprint" "Connector_PinHeader_2.54mm:PinHeader_1x02_P2.54mm_Vertical"
+		(property "Footprint" "Connector_JST:JST_SH_BM02B-SRSS-TB_1x02-1MP_P1.00mm_Vertical"
 			(at 535.94 157.48 0)
 			(hide yes)

Commit message: Removed usb connection components and finished circuit
Parts:
- removed J1: USB_C_Receptacle_USB2.0_14P, Connector_USB:USB_C_Receptacle_G-Switch_GT-USB-7010ASV, symbol Connector:USB_C_Receptacle_USB2.0_14P
- removed Q10: IRLML2246, Package_TO_SOT_SMD:SOT-23, symbol Transistor_FET:IRLML6401
- removed Q9: MMBT3904, Package_TO_SOT_SMD:SOT-23, symbol Transistor_BJT:MMBT3904
- removed R24, R25: 1.3k, Resistor_SMD:R_0603_1608Metric_Pad0.98x0.95mm_HandSolder, symbol Device:R_US
- removed R26: 33k, Resistor_SMD:R_0603_1608Metric_Pad0.98x0.95mm_HandSolder, symbol Device:R_US
- removed R27: 41k, Resistor_SMD:R_0603_1608Metric_Pad0.98x0.95mm_HandSolder, symbol Device:R_US
- removed R28: 100k, Resistor_SMD:R_0603_1608Metric_Pad0.98x0.95mm_HandSolder, symbol Device:R_US
- removed U7: CM1224-02SR, CM1224-02SR:SOT143, symbol CM1224-02SR:CM1224-02SR
- added J5: USB_C_Receptacle_PowerOnly_6P, Connector_USB:USB_C_Receptacle_GCT_USB4125-xx-x-0190_6P_TopMnt_Horizontal, symbol Connector:USB_C_Receptacle_PowerOnly_6P
Connections:
- net 5V USB: now also J5.A9 (VBUS), J5.B9 (VBUS)
- net GND: now also J5.A12 (GND), J5.B12 (GND)
- net at R2.1: now also J5.A5 (CC1)
- net at R1.1: now also J5.B5 (CC2)
- net PA14 USB VBUS: no longer names the net of U5.31 (PA14)
- net TARGET USB N: no longer names the net of U5.45 (PA24)
- net TARGET USB P: no longer names the net of U5.46 (PA25)
Other:
- moved on the sheet: R1, R2
