File: eda/lumi-square/LumiSquare.kicad_sch (KiCad schematic)
At the start: 94 parts, among them J2 Conn_01x12, J3 Conn_01x12, J4 Conn_01x02, J5 USB_C_Receptacle_PowerOnly_6P, J7 FTSH-105-01-X-DV-P-K-X, Q1 IRLML6244, Q15 TSM680P06CH, Q16 TSM680P06CH, Q17 TSM680P06CH, Q18 TSM680P06CH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

Commit message: Fixed warnings
Parts:
- J4: footprint Connector_JST:JST_SH_BM02B-SRSS-TB_1x02-1MP_P1.00mm_Vertical -> Connector_JST:JST_SH_SM02B-SRSS-TB_1x02-1MP_P1.00mm_Horizontal
Changed lines of the file:
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@@
 			)
 		)
-		(property "Footprint" "Connector_JST:JST_SH_BM02B-SRSS-TB_1x02-1MP_P1.00mm_Vertical"
+		(property "Footprint" "Connector_JST:JST_SH_SM02B-SRSS-TB_1x02-1MP_P1.00mm_Horizontal"
 			(at 168.91 189.23 0)
 			(hide yes)

Commit message: Fixed header positions
Parts:
- C10, C8, C9: footprint Capacitor_THT:CP_Radial_D6.3mm_P2.50mm -> Capacitor_Tantalum_SMD:CP_EIA-6032-28_Kemet-C_HandSolder
Changed lines of the file:
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@@
 			)
 		)
-		(property "Footprint" "Capacitor_THT:CP_Radial_D6.3mm_P2.50mm"
+		(property "Footprint" "Capacitor_Tantalum_SMD:CP_EIA-6032-28_Kemet-C_HandSolder"
 			(at 395.9352 57.15 0)
 			(hide yes)
@@
 			)
 		)
-		(property "Footprint" "Capacitor_THT:CP_Radial_D6.3mm_P2.50mm"
+		(property "Footprint" "Capacitor_Tantalum_SMD:CP_EIA-6032-28_Kemet-C_HandSolder"
 			(at 367.9952 57.15 0)
 			(hide yes)
@@
 			)
 		)
-		(property "Footprint" "Capacitor_THT:CP_Radial_D6.3mm_P2.50mm"
+		(property "Footprint" "Capacitor_Tantalum_SMD:CP_EIA-6032-28_Kemet-C_HandSolder"
 			(at 381.9652 57.15 0)
 			(hide yes)

Commit message: Added test points
Parts:
- added H1, H2, H3, H4: MountingHole, MountingHole:MountingHole_2.2mm_M2_DIN965_Pad, symbol Mechanical:MountingHole
- added J1, J10, J11, J12, J13, J14, J15, J16, J17, J6, J8, J9: Conn_01x01, TestPoint:TestPoint_Pad_D1.0mm, symbol Connector_Generic:Conn_01x01
Connections:
- net +3.3V Main: now also J9.1 (Pin_1)
- net 5.3V Out: now also J1.1 (Pin_1)
- net Difficulty Btn: now also J12.1 (Pin_1)
- net GND: now also J8.1 (Pin_1)
- net MCU RX: now also J14.1 (Pin_1)
- net MCU TX: now also J13.1 (Pin_1)
- net Next Btn: now also J11.1 (Pin_1)
- net Previous Btn: now also J10.1 (Pin_1)
- net SPI CLK: now also J16.1 (Pin_1)
- net SPI Dout: now also J15.1 (Pin_1)
- net SPI Latch: now also J17.1 (Pin_1)
- net at Q1.3 (D), R6.2, U2.1 (RESET)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: now also J6.1 (Pin_1)
Other:
- note added: "Mounting Holes"
